File: Schematics/Address_decoder_extended/Address_decoder_extended.sch (KiCad schematic (older format))
At the start: 7 parts, among them J1 Address bus, J2 Clock, J3 ROM select, J4 RAM select, J5 VIA1 select, U1 74HC00, U2 74HC04

Commit message: Added schematic for extended address decoder
Parts:
- removed U2: 74HC04, symbol 74xx:74HC04
- added J6: VIA1 select, symbol Connector:Conn_01x06_Female
- added U2: 7402, symbol 74xx:7402
Connections:
- net labels added: VIA2_CS1, VIA2_RS0, VIA2_RS1, VIA2_RS2, VIA2_RS3, VIA2_~CS2
- wire segments 45 -> 59
- no-connect marks 9 -> 7
Other:
- moved on the sheet: U1B
Changed lines of the file:
@@
 encoding utf-8
 Sheet 1 1
-Title "Address decoder (basic v2)"
-Date "2019-12-30"
+Title "Address decoder (basic extended)"
+Date "2020-01-02"
 Rev "v01"
 Comp ""
@@
 Text Label 7400 4200 0    50   ~ 0
 VIA1_RS0
-Text Label 4850 3400 0    50   ~ 0
-a15
-Wire Wire Line
-	7200 2900 7850 2900
-$Comp
-L 74xx:74HC00 U1
-U 1 1 5E0C758B
-P 5500 2800
-F 0 "U1" H 5500 3125 50  0000 C CNN
-F 1 "74HC00" H 5500 3034 50  0000 C CNN
-F 2 "" H 5500 2800 50  0001 C CNN
-F 3 "http://www.ti.com/lit/gpn/sn74hc00" H 5500 2800 50  0001 C CNN
-	1    5500 2800
-	1    0    0    -1
-$EndComp
-Entry Wire Line
-	4750 3500 4850 3400
-$Comp
-L 74xx:74HC00 U1
-U 2 1 5E0D5C1A
-P 6300 3500
-F 0 "U1" H 6300 3825 50  0000 C CNN
-F 1 "74HC00" H 6300 3734 50  0000 C CNN
-F 2 "" H 6300 3500 50  0001 C CNN
-F 3 "http://www.ti.com/lit/gpn/sn74hc00" H 6300 3500 50  0001 C CNN
-	2    6300 3500
-	1    0    0    -1
-$EndComp
 Text Label 7100 3900 0    50   ~ 0
 a3
@@
 Wire Wire Line
 	7100 3900 7850 3900
-Text GLabel 5900 3600 0    50   Input ~ 0
-CLK
-Wire Wire Line
-	5900 3600 6000 3600
-Wire Wire Line
-	6600 3500 6650 3500
 Text Label 4850 4250 0    50   ~ 0
 a15
@@
 	4750 4350 4850 4250
 Wire Wire Line
-	4850 4250 6000 4250
-Wire Wire Line
-	6000 4050 5800 4050
-Wire Wire Line
 	6600 4150 6800 4150
-Wire Bus Line
-	3800 4450 4750 4450
-Connection ~ 4750 4450
-Wire Bus Line
-	4750 4450 6000 4450
-Text Label 6100 4750 0    50   ~ 0
-a12
-Text Label 6100 4850 0    50   ~ 0
-a11
 Text Label 6100 4950 0    50   ~ 0
 a10
@@
 Text Label 6100 5550 0    50   ~ 0
 a4
-NoConn ~ 6100 4750
-NoConn ~ 6100 4850
 NoConn ~ 6100 4950
 NoConn ~ 6100 5050
@@
 NoConn ~ 6100 5550
 Entry Wire Line
-	6000 4750 6100 4850
-Entry Wire Line
-	6000 4650 6100 4750
-Entry Wire Line
 	6000 4850 6100 4950
 Entry Wire Line
@@
 Wire Bus Line
 	6000 4450 7000 4450
-Wire Wire Line
-	7200 3250 7200 3350
-Wire Wire Line
-	7200 3250 7850 3250
-Wire Wire Line
-	7200 3350 7850 3350
-Wire Wire Line
-	7200 3350 6650 3350
-Wire Wire Line
-	6650 3350 6650 3500
-Connection ~ 7200 3350
-$Comp
-L 74xx:74HC04 U2
-U 1 1 5E0E0C1E
-P 5500 3400
-F 0 "U2" H 5500 3717 50  0000 C CNN
-F 1 "74HC04" H 5500 3626 50  0000 C CNN
-F 2 "" H 5500 3400 50  0001 C CNN
-F 3 "https://assets.nexperia.com/documents/data-sheet/74HC_HCT04.pdf" H 5500 3400 50  0001 C CNN
-	1    5500 3400
-	1    0    0    -1
-$EndComp
-Wire Wire Line
-	5800 2800 7200 2800
-Wire Wire Line
-	5800 3400 6000 3400
-Wire Wire Line
-	4850 3400 5200 3400
-Wire Wire Line
-	7200 2900 7200 2800
-Connection ~ 7200 2800
-Wire Wire Line
-	7200 2800 7850 2800
-Text Label 4850 2700 0    50   ~ 0
-a15
-Text Label 4850 2900 0    50   ~ 0
+Text Label 4850 4150 0    50   ~ 0
 a14
-Wire Wire Line
-	4850 2900 5200 2900
-Wire Wire Line
-	4850 2700 5200 2700
-Entry Wire Line
-	4750 2800 4850 2700
-Entry Wire Line
-	4750 3000 4850 2900
-$Comp
-L 74xx:74HC04 U2
-U 6 1 5E1086B3
-P 5500 4050
-F 0 "U2" H 5500 4367 50  0000 C CNN
-F 1 "74HC04" H 5500 4276 50  0000 C CNN
-F 2 "" H 5500 4050 50  0001 C CNN
-F 3 "https://assets.nexperia.com/documents/data-sheet/74HC_HCT04.pdf" H 5500 4050 50  0001 C CNN
-	6    5500 4050
-	1    0    0    -1
-$EndComp
-Text Label 4850 4050 0    50   ~ 0
-a14
-Entry Wire Line
-	4750 4150 4850 4050
-Wire Wire Line
-	4850 4050 5200 4050
+Entry Wire Line
+	4750 4050 4850 3950
+Wire Wire Line
+	4850 4150 5200 4150
 Wire Wire Line
 	6800 4150 6800 3550
@@
 	7000 3800 7100 3700
 Text Label 7100 3700 0    50   ~ 0
+a12
+Wire Wire Line
+	7100 3700 7850 3700
+Connection ~ 4750 4450
+Wire Bus Line
+	4750 4450 6000 4450
+Wire Bus Line
+	3800 4450 4750 4450
+Wire Wire Line
+	5100 3250 5100 3150
+Wire Wire Line
+	5100 3350 5200 3350
+Wire Wire Line
+	5200 3150 5100 3150
+$Comp
+L 74xx:74HC00 U1
+U 1 1 5E0E6448
+P 5500 3250
+F 0 "U1" H 5500 3575 50  0000 C CNN
+F 1 "74HC00" H 5500 3484 50  0000 C CNN
+F 2 "" H 5500 3250 50  0001 C CNN
+F 3 "http://www.ti.com/lit/gpn/sn74hc00" H 5500 3250 50  0001 C CNN
+	1    5500 3250
+	1    0    0    -1
+$EndComp
+Wire Wire Line
+	4850 3250 5100 3250
+Wire Wire Line
+	5800 3250 5900 3250
+Wire Wire Line
+	6600 3350 7200 3350
+Wire Wire Line
+	5900 3450 6000 3450
+Text GLabel 5900 3450 0    50   Input ~ 0
+CLK
+$Comp
+L 74xx:74HC00 U1
+U 2 1 5E0D5C1A
+P 6300 3350
+F 0 "U1" H 6300 3675 50  0000 C CNN
+F 1 "74HC00" H 6300 3584 50  0000 C CNN
+F 2 "" H 6300 3350 50  0001 C CNN
+F 3 "http://www.ti.com/lit/gpn/sn74hc00" H 6300 3350 50  0001 C CNN
+	2    6300 3350
+	1    0    0    -1
+$EndComp
+Entry Wire Line
+	4750 3350 4850 3250
+Text Label 4850 3250 0    50   ~ 0
+a15
+Wire Wire Line
+	7200 3350 7850 3350
+Wire Wire Line
+	7200 3350 7200 3250
+Wire Wire Line
+	7200 3250 7850 3250
+Wire Wire Line
+	5900 3250 5900 2900
+Connection ~ 5900 3250
+Wire Wire Line
+	5900 3250 6000 3250
+$Comp
+L 74xx:7402 U2
+U 4 1 5E130222
+P 5500 4050
+F 0 "U2" H 5500 4375 50  0000 C CNN
+F 1 "7402" H 5500 4284 50  0000 C CNN
+F 2 "" H 5500 4050 50  0001 C CNN
+F 3 "http://www.ti.com/lit/gpn/sn7402" H 5500 4050 50  0001 C CNN
+	4    5500 4050
+	1    0    0    -1
+$EndComp
+Text Label 4850 3950 0    50   ~ 0
 a13
 Wire Wire Line
-	7100 3700 7850 3700
+	5200 3950 4850 3950
+Wire Wire Line
+	4850 4250 6000 4250
+Wire Wire Line
+	5800 4050 5900 4050
+Connection ~ 7200 3350
+Connection ~ 5100 3250
+Wire Wire Line
+	5100 3250 5100 3350
+Wire Wire Line
+	5900 2900 7850 2900
+Entry Wire Line
+	4750 4250 4850 4150
+Wire Wire Line
+	5900 4050 5900 3650
+Wire Wire Line
+	5900 3650 6650 3650
+Wire Wire Line
+	6650 3650 6650 2800
+Connection ~ 5900 4050
+Wire Wire Line
+	5900 4050 6000 4050
+Wire Wire Line
+	6650 2800 7850 2800
+$Comp
+L Connector:Conn_01x06_Female J6
+U 1 1 5E0FB26B
+P 8050 4800
+F 0 "J6" H 7400 5150 50  0000 L CNN
+F 1 "VIA1 select" H 7650 5150 50  0000 L CNN
+F 2 "" H 8050 4800 50  0001 C CNN
+F 3 "~" H 8050 4800 50  0001 C CNN
+	1    8050 4800
+	1    0    0    -1
+$EndComp
+Text Label 7400 4600 0    50   ~ 0
+VIA2_CS1
+Text Label 7400 4700 0    50   ~ 0
+VIA2_~CS2
+Text Label 7400 4800 0    50   ~ 0
+VIA2_RS3
+Text Label 7400 4900 0    50   ~ 0
+VIA2_RS2
+Text Label 7400 5000 0    50   ~ 0
+VIA2_RS1
+Text Label 7400 5100 0    50   ~ 0
+VIA2_RS0
+Text Label 7100 4600 0    50   ~ 0
+a11
+Wire Wire Line
+	7100 4600 7850 4600
+Text Label 7100 4800 0    50   ~ 0
+a3
+Text Label 7100 4900 0    50   ~ 0
+a2
+Text Label 7100 5000 0    50   ~ 0
+a1
+Text Label 7100 5100 0    50   ~ 0
+a0
+Wire Wire Line
+	7100 5100 7850 5100
+Wire Wire Line
+	7100 5000 7850 5000
+Wire Wire Line
+	7100 4900 7850 4900
+Wire Wire Line
+	7100 4800 7850 4800
+Entry Wire Line
+	7000 5000 7100 5100
+Entry Wire Line
+	7000 4900 7100 5000
+Entry Wire Line
+	7000 4800 7100 4900
+Entry Wire Line
+	7000 4700 7100 4800
+Entry Wire Line
+	7000 4500 7100 4600
+Connection ~ 7000 4450
+Wire Wire Line
+	7300 4700 7300 4350
+Wire Wire Line
+	7300 4350 6800 4350
+Wire Wire Line
+	6800 4350 6800 4150
+Wire Wire Line
+	7300 4700 7850 4700
 Wire Bus Line
 	7000 3800 7000 4450
 Wire Bus Line
-	4750 2800 4750 4450
+	4750 3350 4750 4450
 Wire Bus Line
 	6000 4450 6000 5450
 Wire Bus Line
+	7000 4450 7000 5000
+Wire Bus Line
 	3800 2900 3800 4450
+Connection ~ 6800 4150
 $EndSCHEMATC
