File: Schematics/65C02_Computer/6502_IO.sch (KiCad schematic (older format))
At the start: 25 parts, among them J3 USB_B_Micro, J4 LCD Connector, J5 VIA2PA, J6 VIA2PB, J7 Mini-DIN-6, U10 ATtiny4313-PU, U11 65C22S, U12 65C22S, U5 65C51N, U6 FT230XS, X2 1.8432MHz

Commit message: Redesign in progress
Parts:
- added J10: USB_B, Connector_USB:USB_B_OST_USB-B1HSxx_Horizontal, symbol Connector:USB_B
- added J8: Optional UART Port, Connector_PinSocket_2.54mm:PinSocket_1x06_P2.54mm_Vertical, symbol Connector:Conn_01x06_Female
- added J9: Power Connector, Connector_BarrelJack:BarrelJack_Horizontal, symbol Connector:Barrel_Jack
Connections:
- net +5V: now also J10.1 (VBUS), J8.6 (Pin_6), J9.1
- net GND: now also J10.4 (GND), J8.5 (Pin_5), J9.2
- net RxD: now also J8.2 (Pin_2)
- net TxD: now also J8.1 (Pin_1)
- net USBD+: now also C9.1, J3.3 (D+), J10.3 (D+); no longer U6.8 (USBD+)
- net USBD-: now also C10.1, J3.2 (D-), J10.2 (D-); no longer U6.9 (USBD-)
- net ~CTS: now also J8.4 (Pin_4)
- net ~RTS: now also J8.3 (Pin_3)
- new net: R5.2, U6.8 (USBD+)
- new net: R4.2, U6.9 (USBD-)
- no-connect marks 16 -> 17
Other:
- moved on the sheet: R4, R5
Changed lines of the file:
@@
 Wire Wire Line
 	3750 1600 4100 1600
-Text GLabel 4000 2200 3    50   BiDi ~ 0
+Text GLabel 4000 2600 3    50   BiDi ~ 0
 USBD+
-Text GLabel 5300 2200 3    50   BiDi ~ 0
+Text GLabel 5300 2600 3    50   BiDi ~ 0
 USBD-
 Wire Wire Line
 	3750 1050 4800 1050
-Wire Wire Line
-	4000 2100 4000 2200
 Wire Wire Line
 	4000 2100 4100 2100
@@
 Wire Wire Line
 	1950 1950 1550 1950
-Wire Wire Line
-	2000 1350 1950 1350
 Connection ~ 1950 1350
-Wire Wire Line
-	2300 1350 2450 1350
-Wire Wire Line
-	2300 1450 2450 1450
-Wire Wire Line
-	2000 1450 1550 1450
 Connection ~ 1550 1450
 Wire Wire Line
 	5200 2100 5300 2100
-Wire Wire Line
-	5300 2100 5300 2200
 NoConn ~ 4100 2000
 Wire Wire Line
@@
 L Device:R R?
 U 1 1 5F203CE6
-P 2150 1450
+P 5300 2400
 AR Path="/5F203CE6" Ref="R?"  Part="1"
 AR Path="/5F14295C/5F203CE6" Ref="R4"  Part="1"
-F 0 "R4" V 2250 1450 50  0000 C CNN
-F 1 "27" V 2150 1450 50  0000 C CNN
-F 2 "Resistor_THT:R_Axial_DIN0207_L6.3mm_D2.5mm_P7.62mm_Horizontal" V 2080 1450 50  0001 C CNN
-F 3 "~" H 2150 1450 50  0001 C CNN
-	1    2150 1450
-	0    1    1    0
+F 0 "R4" V 5400 2400 50  0000 C CNN
+F 1 "27" V 5300 2400 50  0000 C CNN
+F 2 "Resistor_THT:R_Axial_DIN0207_L6.3mm_D2.5mm_P7.62mm_Horizontal" V 5230 2400 50  0001 C CNN
+F 3 "~" H 5300 2400 50  0001 C CNN
+	1    5300 2400
+	-1   0    0    1
 $EndComp
 $Comp
 L Device:R R?
 U 1 1 5F203CE0
-P 2150 1350
+P 4000 2400
 AR Path="/5F203CE0" Ref="R?"  Part="1"
 AR Path="/5F14295C/5F203CE0" Ref="R5"  Part="1"
-F 0 "R5" V 2050 1350 50  0000 C CNN
-F 1 "27" V 2150 1350 50  0000 C CNN
-F 2 "Resistor_THT:R_Axial_DIN0207_L6.3mm_D2.5mm_P7.62mm_Horizontal" V 2080 1350 50  0001 C CNN
-F 3 "~" H 2150 1350 50  0001 C CNN
-	1    2150 1350
-	0    1    1    0
+F 0 "R5" V 3900 2400 50  0000 C CNN
+F 1 "27" V 4000 2400 50  0000 C CNN
+F 2 "Resistor_THT:R_Axial_DIN0207_L6.3mm_D2.5mm_P7.62mm_Horizontal" V 3930 2400 50  0001 C CNN
+F 3 "~" H 4000 2400 50  0001 C CNN
+	1    4000 2400
+	-1   0    0    1
 $EndComp
 $Comp
@@
 Wire Wire Line
 	6850 5650 6950 5650
+$Comp
+L Connector:Conn_01x06_Female J8
+U 1 1 5E4D0B3D
+P 2850 6100
+F 0 "J8" H 2878 6076 50  0000 L CNN
+F 1 "Optional UART Port" H 2878 5985 50  0000 L CNN
+F 2 "Connector_PinSocket_2.54mm:PinSocket_1x06_P2.54mm_Vertical" H 2850 6100 50  0001 C CNN
+F 3 "~" H 2850 6100 50  0001 C CNN
+	1    2850 6100
+	1    0    0    -1
+$EndComp
+Text GLabel 2550 6000 0    50   Output ~ 0
+RxD
+Text GLabel 2550 5900 0    50   Input ~ 0
+TxD
+Text GLabel 2350 6100 0    50   BiDi ~ 0
+~RTS
+Text GLabel 2550 6200 0    50   BiDi ~ 0
+~CTS
+Text GLabel 2550 6400 0    50   Input ~ 0
++5V
+Text GLabel 2350 6300 0    50   Input ~ 0
+GND
+Wire Wire Line
+	2550 5900 2650 5900
+Wire Wire Line
+	2550 6000 2650 6000
+Wire Wire Line
+	2350 6100 2650 6100
+Wire Wire Line
+	2550 6200 2650 6200
+Wire Wire Line
+	2350 6300 2650 6300
+Wire Wire Line
+	2550 6400 2650 6400
+$Comp
+L Connector:Barrel_Jack J9
+U 1 1 5E59BEED
+P 2550 6900
+F 0 "J9" H 2607 7225 50  0000 C CNN
+F 1 "Power Connector" H 2607 7134 50  0000 C CNN
+F 2 "Connector_BarrelJack:BarrelJack_Horizontal" H 2600 6860 50  0001 C CNN
+F 3 "~" H 2600 6860 50  0001 C CNN
+	1    2550 6900
+	1    0    0    -1
+$EndComp
+Text GLabel 2950 6800 2    50   Input ~ 0
++5V
+Text GLabel 2950 7000 2    50   Input ~ 0
+GND
+Wire Wire Line
+	2950 7000 2850 7000
+Wire Wire Line
+	2950 6800 2850 6800
+$Comp
+L Connector:USB_B J10
+U 1 1 5E5D8CF6
+P 3950 6800
+F 0 "J10" H 4007 7267 50  0000 C CNN
+F 1 "USB_B" H 4007 7176 50  0000 C CNN
+F 2 "Connector_USB:USB_B_OST_USB-B1HSxx_Horizontal" H 4100 6750 50  0001 C CNN
+F 3 " ~" H 4100 6750 50  0001 C CNN
+	1    3950 6800
+	1    0    0    -1
+$EndComp
+Text GLabel 3950 7300 3    50   Input ~ 0
+GND
+Text GLabel 4350 6600 2    50   Input ~ 0
++5V
+Text GLabel 4350 6800 2    50   BiDi ~ 0
+USBD+
+Text GLabel 4350 6900 2    50   BiDi ~ 0
+USBD-
+NoConn ~ 3850 7200
+Wire Wire Line
+	3950 7300 3950 7200
+Wire Wire Line
+	4250 6900 4350 6900
+Wire Wire Line
+	4250 6800 4350 6800
+Wire Wire Line
+	4250 6600 4350 6600
+Wire Wire Line
+	1950 1350 2450 1350
+Wire Wire Line
+	1550 1450 2450 1450
+Wire Wire Line
+	4000 2600 4000 2550
+Wire Wire Line
+	4000 2100 4000 2250
+Wire Wire Line
+	5300 2100 5300 2250
+Wire Wire Line
+	5300 2550 5300 2600
 Wire Bus Line
 	5500 3000 5500 3400

Commit message: PCB RC1
Parts:
- renumbered J4 to J10, J8 to J2, J10 to J4, J9 to J5, J7 to J6, J5 to J8, J6 to J9
Connections:
- net USBD+: now also U6.8 (USBD+); no longer C9.1, J3.3 (D+), J4.3 (D+)
- net USBD-: now also U6.9 (USBD-); no longer C10.1, J3.2 (D-), J4.2 (D-)
- net PUSBD+: now reaches R5.2
- net PUSBD+: now also C9.1, J3.3 (D+), J4.3 (D+); no longer U6.8 (USBD+)
- net PUSBD-: now reaches R4.2
- net PUSBD-: now also C10.1, J3.2 (D-), J4.2 (D-); no longer U6.9 (USBD-)
Other:
- moved on the sheet: J3, R4, R5
Changed lines of the file:
@@
 Sheet 2 2
 Title "65C02 Hobby Computer"
-Date "2020-02-03"
+Date "2020-02-17"
 Rev "v001"
 Comp ""
@@
 Wire Wire Line
 	3750 1600 4100 1600
-Text GLabel 4000 2600 3    50   BiDi ~ 0
+Text GLabel 4000 2200 3    50   BiDi ~ 0
 USBD+
-Text GLabel 5300 2600 3    50   BiDi ~ 0
+Text GLabel 5300 2200 3    50   BiDi ~ 0
 USBD-
 Wire Wire Line
@@
 Wire Wire Line
 	4000 2100 4100 2100
-NoConn ~ 1050 1750
-Wire Wire Line
-	1450 1150 2350 1150
 Wire Wire Line
 	2350 1150 2350 1100
-Wire Wire Line
-	1150 1750 1150 1950
-NoConn ~ 1450 1550
 Text GLabel 2450 1350 2    50   BiDi ~ 0
 USBD+
@@
 USBD-
 Wire Wire Line
-	1450 1350 1950 1350
-Wire Wire Line
 	1450 1450 1550 1450
 Wire Wire Line
 	1550 1850 1550 1950
 Wire Wire Line
-	1550 1950 1150 1950
-Connection ~ 1150 1950
-Wire Wire Line
-	1150 1950 1150 2050
-Wire Wire Line
 	1950 1850 1950 1950
 Wire Wire Line
 	1950 1950 2350 1950
-Connection ~ 1550 1950
 Wire Wire Line
 	1550 1550 1550 1450
@@
 Wire Wire Line
 	1950 1950 1550 1950
-Connection ~ 1950 1350
-Connection ~ 1550 1450
 Wire Wire Line
 	5200 2100 5300 2100
@@
 	2950 1250 2950 1150
 $Comp
-L Connector:Mini-DIN-6 J7
+L Connector:Mini-DIN-6 J6
 U 1 1 5F701D58
 P 9550 2650
-F 0 "J7" H 9550 3017 50  0000 C CNN
+F 0 "J6" H 9550 3017 50  0000 C CNN
 F 1 "Mini-DIN-6" H 9550 2926 50  0000 C CNN
 F 2 "65C02_Computer:mini_din-6" H 9550 2650 50  0001 C CNN
@@
 L power:GND #PWR?
 U 1 1 5F26EEF9
-P 1150 2050
+P 2350 2050
 AR Path="/5F26EEF9" Ref="#PWR?"  Part="1"
 AR Path="/5F14295C/5F26EEF9" Ref="#PWR03"  Part="1"
-F 0 "#PWR03" H 1150 1800 50  0001 C CNN
-F 1 "GND" H 1155 1877 50  0000 C CNN
-F 2 "" H 1150 2050 50  0001 C CNN
-F 3 "" H 1150 2050 50  0001 C CNN
-	1    1150 2050
+F 0 "#PWR03" H 2350 1800 50  0001 C CNN
+F 1 "GND" H 2355 1877 50  0000 C CNN
+F 2 "" H 2350 2050 50  0001 C CNN
+F 3 "" H 2350 2050 50  0001 C CNN
+	1    2350 2050
 	1    0    0    -1
 $EndComp
@@
 L Connector:USB_B_Micro J?
 U 1 1 5F26EEF2
-P 1150 1350
+P 5300 6800
 AR Path="/5F26EEF2" Ref="J?"  Part="1"
 AR Path="/5F14295C/5F26EEF2" Ref="J3"  Part="1"
-F 0 "J3" H 1207 1817 50  0000 C CNN
-F 1 "USB_B_Micro" H 1207 1726 50  0000 C CNN
-F 2 "Connector_USB:USB_Micro-B_Molex-105017-0001" H 1300 1300 50  0001 C CNN
-F 3 "~" H 1300 1300 50  0001 C CNN
-	1    1150 1350
+F 0 "J3" H 5357 7267 50  0000 C CNN
+F 1 "USB_B_Micro" H 5357 7176 50  0000 C CNN
+F 2 "Connector_USB:USB_Micro-B_Molex-105017-0001" H 5450 6750 50  0001 C CNN
+F 3 "~" H 5450 6750 50  0001 C CNN
+	1    5300 6800
 	1    0    0    -1
 $EndComp
@@
 L Device:R R?
 U 1 1 5F203CE6
-P 5300 2400
+P 2150 1450
 AR Path="/5F203CE6" Ref="R?"  Part="1"
 AR Path="/5F14295C/5F203CE6" Ref="R4"  Part="1"
-F 0 "R4" V 5400 2400 50  0000 C CNN
-F 1 "27" V 5300 2400 50  0000 C CNN
-F 2 "Resistor_THT:R_Axial_DIN0207_L6.3mm_D2.5mm_P7.62mm_Horizontal" V 5230 2400 50  0001 C CNN
-F 3 "~" H 5300 2400 50  0001 C CNN
-	1    5300 2400
-	-1   0    0    1
+F 0 "R4" V 2250 1450 50  0000 C CNN
+F 1 "27" V 2150 1450 50  0000 C CNN
+F 2 "Resistor_THT:R_Axial_DIN0207_L6.3mm_D2.5mm_P7.62mm_Horizontal" V 2080 1450 50  0001 C CNN
+F 3 "~" H 2150 1450 50  0001 C CNN
+	1    2150 1450
+	0    1    1    0
 $EndComp
 $Comp
 L Device:R R?
 U 1 1 5F203CE0
-P 4000 2400
+P 2150 1350
 AR Path="/5F203CE0" Ref="R?"  Part="1"
 AR Path="/5F14295C/5F203CE0" Ref="R5"  Part="1"
-F 0 "R5" V 3900 2400 50  0000 C CNN
-F 1 "27" V 4000 2400 50  0000 C CNN
-F 2 "Resistor_THT:R_Axial_DIN0207_L6.3mm_D2.5mm_P7.62mm_Horizontal" V 3930 2400 50  0001 C CNN
-F 3 "~" H 4000 2400 50  0001 C CNN
-	1    4000 2400
-	-1   0    0    1
+F 0 "R5" V 2050 1350 50  0000 C CNN
+F 1 "27" V 2150 1350 50  0000 C CNN
+F 2 "Resistor_THT:R_Axial_DIN0207_L6.3mm_D2.5mm_P7.62mm_Horizontal" V 2080 1350 50  0001 C CNN
+F 3 "~" H 2150 1350 50  0001 C CNN
+	1    2150 1350
+	0    1    1    0
 $EndComp
 $Comp
@@
 	1050 3000 3100 3000
 $Comp
-L Connector:Conn_01x16_Female J4
+L Connector:Conn_01x16_Female J10
 U 1 1 5FB15958
 P 6650 4150
-F 0 "J4" H 6678 4126 50  0000 L CNN
+F 0 "J10" H 6678 4126 50  0000 L CNN
 F 1 "LCD Connector" H 6678 4035 50  0000 L CNN
 F 2 "Connector_PinSocket_2.54mm:PinSocket_1x16_P2.54mm_Vertical" H 6650 4150 50  0001 C CNN
@@
 v2pa9
 $Comp
-L Connector:Conn_01x12_Male J5
+L Connector:Conn_01x12_Male J8
 U 1 1 5FD88768
 P 8150 3750
-F 0 "J5" V 8100 3800 50  0000 L CNN
+F 0 "J8" H 8200 4400 50  0000 L CNN
 F 1 "VIA2PA" V 8100 3500 50  0000 L CNN
 F 2 "Connector_PinHeader_2.54mm:PinHeader_1x12_P2.54mm_Vertical" H 8150 3750 50  0001 C CNN
@@
 	7550 4050 7650 4150
 $Comp
-L Connector:Conn_01x12_Male J6
+L Connector:Conn_01x12_Male J9
 U 1 1 5FEAF969
 P 8150 5150
-F 0 "J6" V 8100 5200 50  0000 L CNN
+F 0 "J9" H 8200 5800 50  0000 L CNN
 F 1 "VIA2PB" V 8100 4900 50  0000 L CNN
 F 2 "Connector_PinHeader_2.54mm:PinHeader_1x12_P2.54mm_Vertical" H 8150 5150 50  0001 C CNN
@@
 	6850 5650 6950 5650
 $Comp
-L Connector:Conn_01x06_Female J8
+L Connector:Conn_01x06_Female J2
 U 1 1 5E4D0B3D
 P 2850 6100
-F 0 "J8" H 2878 6076 50  0000 L CNN
+F 0 "J2" H 2878 6076 50  0000 L CNN
 F 1 "Optional UART Port" H 2878 5985 50  0000 L CNN
 F 2 "Connector_PinSocket_2.54mm:PinSocket_1x06_P2.54mm_Vertical" H 2850 6100 50  0001 C CNN
@@
 	2550 6400 2650 6400
 $Comp
-L Connector:Barrel_Jack J9
+L Connector:Barrel_Jack J5
 U 1 1 5E59BEED
 P 2550 6900
-F 0 "J9" H 2607 7225 50  0000 C CNN
+F 0 "J5" H 2607 7225 50  0000 C CNN
 F 1 "Power Connector" H 2607 7134 50  0000 C CNN
 F 2 "Connector_BarrelJack:BarrelJack_Horizontal" H 2600 6860 50  0001 C CNN
@@
 	2950 6800 2850 6800
 $Comp
-L Connector:USB_B J10
+L Connector:USB_B J4
 U 1 1 5E5D8CF6
 P 3950 6800
-F 0 "J10" H 4007 7267 50  0000 C CNN
+F 0 "J4" H 4007 7267 50  0000 C CNN
 F 1 "USB_B" H 4007 7176 50  0000 C CNN
 F 2 "Connector_USB:USB_B_OST_USB-B1HSxx_Horizontal" H 4100 6750 50  0001 C CNN
@@
 +5V
 Text GLabel 4350 6800 2    50   BiDi ~ 0
-USBD+
+PUSBD+
 Text GLabel 4350 6900 2    50   BiDi ~ 0
-USBD-
+PUSBD-
 NoConn ~ 3850 7200
 Wire Wire Line
@@
 	4250 6600 4350 6600
 Wire Wire Line
-	1950 1350 2450 1350
-Wire Wire Line
-	1550 1450 2450 1450
-Wire Wire Line
-	4000 2600 4000 2550
-Wire Wire Line
-	4000 2100 4000 2250
-Wire Wire Line
-	5300 2100 5300 2250
-Wire Wire Line
-	5300 2550 5300 2600
+	4000 2100 4000 2200
+Wire Wire Line
+	5300 2100 5300 2200
+Wire Wire Line
+	1450 1350 1950 1350
+Connection ~ 1950 1350
+Wire Wire Line
+	1950 1350 2000 1350
+Wire Wire Line
+	2300 1350 2450 1350
+Wire Wire Line
+	2450 1450 2300 1450
+Wire Wire Line
+	2000 1450 1550 1450
+Connection ~ 1550 1450
+Text GLabel 5700 6600 2    50   Input ~ 0
++5V
+Text GLabel 5300 7300 3    50   Input ~ 0
+GND
+NoConn ~ 5200 7200
+Wire Wire Line
+	5700 6600 5600 6600
+Wire Wire Line
+	5300 7300 5300 7200
+NoConn ~ 5600 7000
+Text GLabel 5700 6800 2    50   BiDi ~ 0
+PUSBD+
+Text GLabel 5700 6900 2    50   BiDi ~ 0
+PUSBD-
+Wire Wire Line
+	5700 6900 5600 6900
+Wire Wire Line
+	5600 6800 5700 6800
+Wire Wire Line
+	2350 2050 2350 1950
+Text GLabel 1450 1350 0    50   BiDi ~ 0
+PUSBD+
+Text GLabel 1450 1450 0    50   BiDi ~ 0
+PUSBD-
 Wire Bus Line
 	5500 3000 5500 3400

Commit message: PCB RC2 - updated FT230XS footprint
Parts:
- U6: footprint Package_SO:SSOP-16_4.4x5.2mm_P0.65mm -> Package_SO:SSOP-16_3.9x4.9mm_P0.635mm
Changed lines of the file:
@@
 F 0 "U6" H 4650 2365 50  0000 C CNN
 F 1 "FT230XS" H 4650 2274 50  0000 C CNN
-F 2 "Package_SO:SSOP-16_4.4x5.2mm_P0.65mm" H 4650 2250 50  0001 C CNN
+F 2 "Package_SO:SSOP-16_3.9x4.9mm_P0.635mm" H 4650 2250 50  0001 C CNN
 F 3 "https://www.ftdichip.com/Support/Documents/DataSheets/ICs/DS_FT230X.pdf" H 4650 1750 50  0001 C CNN
 	1    4650 1750

Commit message: PCB RC4 - added longer pads to SSOP chip
Parts:
- U6: footprint Package_SO:SSOP-16_3.9x4.9mm_P0.635mm -> 65C02_Computer:SSOP-16_3.9x4.9mm_P0.635mm_long_pads
Changed lines of the file:
@@
 F 0 "U6" H 4650 2365 50  0000 C CNN
 F 1 "FT230XS" H 4650 2274 50  0000 C CNN
-F 2 "Package_SO:SSOP-16_3.9x4.9mm_P0.635mm" H 4650 2250 50  0001 C CNN
+F 2 "65C02_Computer:SSOP-16_3.9x4.9mm_P0.635mm_long_pads" H 4650 2250 50  0001 C CNN
 F 3 "https://www.ftdichip.com/Support/Documents/DataSheets/ICs/DS_FT230X.pdf" H 4650 1750 50  0001 C CNN
 	1    4650 1750
