File: Schematics/Blog/Blog.sch (KiCad schematic (older format))
At the start: 14 parts, among them U1 74HC00, U10 74AC32, U11 74HC74, U12 74AC32, U13 74AC08, U14 74AC74, U2 74HC04, U3 74HC32, U4 74HC08, U5 74HC04, U6 74AC32, U7 74AC08, U8 74HC04, U9 74AC74

Commit message: Drafted four schematics for RDY experiments
Changed lines of the file:
@@
 $Descr A4 11693 8268
 encoding utf-8
-Sheet 1 2
+Sheet 1 5
 Title ""
 Date ""
@@
 	4100 5750 4200 5750
 $Sheet
-S 5450 6900 500  150
+S 7400 5000 500  150
 U 60398E8A
 F0 "RDY input" 50
 F1 "RDY input.sch" 50
 $EndSheet
+$Sheet
+S 7400 5400 500  150
+U 603BD881
+F0 "RDY input 2" 50
+F1 "RDY input 2.sch" 50
+$EndSheet
+$Sheet
+S 7400 5800 500  150
+U 604066AD
+F0 "RDY input 3" 50
+F1 "RDY input 3.sch" 50
+$EndSheet
+$Sheet
+S 7400 6200 500  150
+U 60437255
+F0 "RDY input 4" 50
+F1 "RDY input 4.sch" 50
+$EndSheet
 $EndSCHEMATC
