File: Schematics/OpAmp/inverting_right.sch (KiCad schematic (older format))
At the start: 0 parts

Commit message: Added article about adjustable load
Parts:
- added R1, R3: 47K, symbol Device:R
- added R2, R4, R5: 10K, symbol Device:R
- added R6: 1K, symbol Device:R
- added RV1: 10K, symbol Device:R_POT
- added TP1: V1, symbol Connector:TestPoint
- added TP2: Vout, symbol Connector:TestPoint
- added TP3: V2, symbol Connector:TestPoint
- added U1: LM358, symbol Amplifier_Operational:LM358
Connections:
- new net: R1.2, RV1.1
- new net: R3.1, RV1.3
- new net: RV1.2, TP1.1, U1.2 (-)
- new net: R2.2, R4.1, TP3.1, U1.5 (+)
- new net: R5.1, TP2.1, U1.7
- new net: R5.2, R6.1, U1.6 (-)
- new net: R6.2, U1.1, U1.3 (+)
- new net +5V: R1.1, R2.1
- new net GND: R3.2, R4.2
