File: Schematics/DB6502_proto/ports.sch (KiCad schematic (older format))
At the start: 20 parts, among them J1 Power plug, J10 System Bus, J2 Controls, J3 AVR ISP, J4 Debug USB, J5 JPR, J6 Debug UART, J7 UART A, J8 UART B, J9 I/O Bus

Commit message: Small fixes on PCB
Parts:
- J10: footprint Connector_PinSocket_2.54mm:PinSocket_1x32_P2.54mm_Vertical -> Connector_PinSocket_2.54mm:PinSocket_1x40_P2.54mm_Vertical; symbol Connector:Conn_01x32_Female -> Connector:Conn_01x40_Female
Connections:
- net labels added: 6502_RDY_IN
- wire segments 275 -> 271
Changed lines of the file:
@@
 $EndDescr
 $Comp
-L Connector:Conn_01x32_Female J10
+L Connector:Conn_01x40_Female J10
 U 1 1 6014BD0C
-P 4700 6200
-F 0 "J10" H 4728 6176 50  0000 L CNN
-F 1 "System Bus" H 4728 6085 50  0000 L CNN
-F 2 "Connector_PinSocket_2.54mm:PinSocket_1x32_P2.54mm_Vertical" H 4700 6200 50  0001 C CNN
-F 3 "~" H 4700 6200 50  0001 C CNN
-	1    4700 6200
+P 4300 6200
+F 0 "J10" H 4328 6176 50  0000 L CNN
+F 1 "System Bus" H 4328 6085 50  0000 L CNN
+F 2 "Connector_PinSocket_2.54mm:PinSocket_1x40_P2.54mm_Vertical" H 4300 6200 50  0001 C CNN
+F 3 "~" H 4300 6200 50  0001 C CNN
+	1    4300 6200
 	0    -1   -1   0
 $EndComp
+Text Label 2400 6600 1    50   ~ 0
+a0
+Text Label 2500 6600 1    50   ~ 0
+a1
+Text Label 2600 6600 1    50   ~ 0
+a2
+Text Label 2700 6600 1    50   ~ 0
+a3
+Text Label 2800 6600 1    50   ~ 0
+a4
+Text Label 2900 6600 1    50   ~ 0
+a5
+Text Label 3000 6600 1    50   ~ 0
+a6
+Text Label 3100 6600 1    50   ~ 0
+a7
 Text Label 3200 6600 1    50   ~ 0
-a0
+a8
 Text Label 3300 6600 1    50   ~ 0
-a1
+a9
 Text Label 3400 6600 1    50   ~ 0
-a2
+a10
 Text Label 3500 6600 1    50   ~ 0
-a3
+a11
 Text Label 3600 6600 1    50   ~ 0
-a4
+a12
 Text Label 3700 6600 1    50   ~ 0
-a5
+a13
 Text Label 3800 6600 1    50   ~ 0
-a6
+a14
 Text Label 3900 6600 1    50   ~ 0
-a7
+a15
+Wire Wire Line
+	2400 6600 2400 6400
+Wire Wire Line
+	2500 6600 2500 6400
+Wire Wire Line
+	2600 6600 2600 6400
+Wire Wire Line
+	2700 6600 2700 6400
+Wire Wire Line
+	2800 6600 2800 6400
+Wire Wire Line
+	2900 6600 2900 6400
+Wire Wire Line
+	3000 6600 3000 6400
+Wire Wire Line
+	3100 6600 3100 6400
+Wire Wire Line
+	3200 6600 3200 6400
+Wire Wire Line
+	3300 6600 3300 6400
+Wire Wire Line
+	3400 6600 3400 6400
+Wire Wire Line
+	3500 6600 3500 6400
+Wire Wire Line
+	3600 6600 3600 6400
+Wire Wire Line
+	3700 6600 3700 6400
+Wire Wire Line
+	3800 6600 3800 6400
+Wire Wire Line
+	3900 6600 3900 6400
+Entry Wire Line
+	2300 6700 2400 6600
+Entry Wire Line
+	2400 6700 2500 6600
+Entry Wire Line
+	2500 6700 2600 6600
+Entry Wire Line
+	2600 6700 2700 6600
+Entry Wire Line
+	2700 6700 2800 6600
+Entry Wire Line
+	2800 6700 2900 6600
+Entry Wire Line
+	2900 6700 3000 6600
+Entry Wire Line
+	3000 6700 3100 6600
+Entry Wire Line
+	3100 6700 3200 6600
+Entry Wire Line
+	3200 6700 3300 6600
+Entry Wire Line
+	3300 6700 3400 6600
+Entry Wire Line
+	3400 6700 3500 6600
+Entry Wire Line
+	3500 6700 3600 6600
+Entry Wire Line
+	3600 6700 3700 6600
+Entry Wire Line
+	3700 6700 3800 6600
+Entry Wire Line
+	3800 6700 3900 6600
+Text GLabel 3800 6800 3    50   BiDi ~ 0
+a[0..15]
+Wire Bus Line
+	3800 6800 3800 6700
 Text Label 4000 6600 1    50   ~ 0
-a8
+d0
 Text Label 4100 6600 1    50   ~ 0
-a9
+d1
 Text Label 4200 6600 1    50   ~ 0
-a10
+d2
 Text Label 4300 6600 1    50   ~ 0
-a11
+d3
 Text Label 4400 6600 1    50   ~ 0
-a12
+d4
 Text Label 4500 6600 1    50   ~ 0
-a13
+d5
 Text Label 4600 6600 1    50   ~ 0
-a14
+d6
 Text Label 4700 6600 1    50   ~ 0
-a15
-Wire Wire Line
-	3200 6600 3200 6400
-Wire Wire Line
-	3300 6600 3300 6400
-Wire Wire Line
-	3400 6600 3400 6400
-Wire Wire Line
-	3500 6600 3500 6400
-Wire Wire Line
-	3600 6600 3600 6400
-Wire Wire Line
-	3700 6600 3700 6400
-Wire Wire Line
-	3800 6600 3800 6400
-Wire Wire Line
-	3900 6600 3900 6400
+d7
 Wire Wire Line
 	4000 6600 4000 6400
@@
 Wire Wire Line
 	4700 6600 4700 6400
-Entry Wire Line
-	3100 6700 3200 6600
-Entry Wire Line
-	3200 6700 3300 6600
-Entry Wire Line
-	3300 6700 3400 6600
-Entry Wire Line
-	3400 6700 3500 6600
-Entry Wire Line
-	3500 6700 3600 6600
-Entry Wire Line
-	3600 6700 3700 6600
-Entry Wire Line
-	3700 6700 3800 6600
-Entry Wire Line
-	3800 6700 3900 6600
 Entry Wire Line
 	3900 6700 4000 6600
@@
 	4600 6700 4700 6600
 Text GLabel 4600 6800 3    50   BiDi ~ 0
-a[0..15]
+d[0..7]
 Wire Bus Line
 	4600 6800 4600 6700
-Text Label 4800 6600 1    50   ~ 0
-d0
-Text Label 4900 6600 1    50   ~ 0
-d1
-Text Label 5000 6600 1    50   ~ 0
-d2
-Text Label 5100 6600 1    50   ~ 0
-d3
-Text Label 5200 6600 1    50   ~ 0
-d4
-Text Label 5300 6600 1    50   ~ 0
-d5
-Text Label 5400 6600 1    50   ~ 0
-d6
-Text Label 5500 6600 1    50   ~ 0
-d7
-Wire Wire Line
-	4800 6600 4800 6400
-Wire Wire Line
-	4900 6600 4900 6400
-Wire Wire Line
-	5000 6600 5000 6400
-Wire Wire Line
-	5100 6600 5100 6400
-Wire Wire Line
-	5200 6600 5200 6400
-Wire Wire Line
-	5300 6600 5300 6400
-Wire Wire Line
-	5400 6600 5400 6400
-Wire Wire Line
-	5500 6600 5500 6400
-Entry Wire Line
-	4700 6700 4800 6600
-Entry Wire Line
-	4800 6700 4900 6600
-Entry Wire Line
-	4900 6700 5000 6600
-Entry Wire Line
-	5000 6700 5100 6600
-Entry Wire Line
-	5100 6700 5200 6600
-Entry Wire Line
-	5200 6700 5300 6600
-Entry Wire Line
-	5300 6700 5400 6600
-Entry Wire Line
-	5400 6700 5500 6600
-Text GLabel 5400 6800 3    50   BiDi ~ 0
-d[0..7]
-Wire Bus Line
-	5400 6800 5400 6700
 Text Label 2750 1700 0    50   ~ 0
 d0
@@
 Entry Wire Line
 	2650 2300 2750 2400
-Text GLabel 6350 1100 1    50   Input ~ 0
-SYNC
-Text GLabel 6200 1100 1    50   Input ~ 0
-~ML
-Text GLabel 6050 1100 1    50   Input ~ 0
-~VP
-Text GLabel 5900 1100 1    50   Output ~ 0
-6502_RDY
-Text GLabel 5750 1100 1    50   Output ~ 0
+Text GLabel 5750 1100 1    50   Input ~ 0
 BE
-Text GLabel 5600 1100 1    50   Output ~ 0
+Text GLabel 5600 1100 1    50   Input ~ 0
 ~IRQ
 Text GLabel 5450 1100 1    50   Output ~ 0
@@
 Text GLabel 4850 1100 1    50   Input ~ 0
 R~W
-Text GLabel 6500 1100 1    50   Output ~ 0
-~6502_RES
 Wire Wire Line
 	5150 2100 6850 2100
@@
 Wire Wire Line
 	6200 6650 6400 6650
-Text GLabel 2950 4900 0    50   Input ~ 0
-GND
-Text GLabel 2950 4800 0    50   Input ~ 0
-+5V
-Wire Wire Line
-	2950 4800 3050 4800
-Wire Wire Line
-	2950 4900 3050 4900
+Text GLabel 6400 7550 2    50   Input ~ 0
+6502_CLK
+Wire Wire Line
+	6400 7100 5900 7100
+Wire Wire Line
+	5900 7100 5900 6400
 Text GLabel 6400 7100 2    50   Input ~ 0
-6502_CLK
-Wire Wire Line
-	6400 7100 5900 7100
-Wire Wire Line
-	5900 7100 5900 6400
+R~W
+Wire Wire Line
+	6400 7250 5800 7250
+Wire Wire Line
+	5800 7250 5800 6400
 Text GLabel 6400 7250 2    50   Input ~ 0
-R~W
-Wire Wire Line
-	6400 7250 5800 7250
-Wire Wire Line
-	5800 7250 5800 6400
-Text GLabel 6400 7400 2    50   Input ~ 0
 ~6502_RES
 Wire Wire Line
@@
 Wire Wire Line
 	1200 3700 3050 3700
-Text GLabel 1050 4600 3    50   Input ~ 0
+Text GLabel 1200 4600 3    50   Input ~ 0
 ~6502_RES
 Wire Wire Line
@@
 Wire Wire Line
 	1050 3600 3050 3600
-Text GLabel 6400 7550 2    50   Input ~ 0
+Text GLabel 6400 7400 2    50   Input ~ 0
 SYNC
 Wire Wire Line
@@
 Text GLabel 4750 5000 3    50   Output ~ 0
 6502_RDY
-Text GLabel 6750 5000 3    50   Input ~ 0
-GND
-Text GLabel 6650 5000 3    50   Input ~ 0
-+5V
 Wire Wire Line
 	1500 4600 1500 3900
@@
 Wire Wire Line
 	8750 3400 8850 3400
-Text GLabel 10250 3250 2    50   Input ~ 0
+Text GLabel 10250 3250 2    50   Output ~ 0
 VBUS_SENSE
 Wire Wire Line
@@
 Wire Wire Line
 	2950 1000 3050 1000
-Text GLabel 1200 4600 3    50   Output ~ 0
+Text GLabel 1350 4600 3    50   Output ~ 0
 ~VIA2_IRQ
-Text GLabel 1350 4600 3    50   Output ~ 0
+Text GLabel 1500 4600 3    50   Output ~ 0
 ~EXT_IRQ
 Wire Wire Line
@@
 ~PLD_RD
 Text GLabel 4100 5000 3    50   Input ~ 0
+RAM2_~CS
+Text GLabel 4100 1100 1    50   Input ~ 0
 RAM1_~CS
-Text GLabel 4100 1100 1    50   Input ~ 0
-RAM2_~CS
 Text GLabel 4250 1100 1    50   Input ~ 0
 ROM_~CS
@@
 Wire Wire Line
 	5600 4200 6850 4200
-Wire Wire Line
-	6750 5000 6750 4900
-Wire Wire Line
-	6750 4900 6850 4900
-Wire Wire Line
-	6650 5000 6650 4800
-Wire Wire Line
-	6650 4800 6850 4800
-Text GLabel 1500 4600 3    50   Output ~ 0
+Text GLabel 1650 4600 3    50   Output ~ 0
 ~NMI
+Text GLabel 6500 1100 1    50   Input ~ 0
+~6502_RES
+Text GLabel 6050 1100 1    50   Input ~ 0
+~VP
+Text GLabel 6200 1100 1    50   Input ~ 0
+~ML
+Text GLabel 6350 1100 1    50   Input ~ 0
+SYNC
+Text GLabel 1050 4600 3    50   Input ~ 0
+~6502_CLK
+Text GLabel 6400 7700 2    50   Input ~ 0
+~6502_CLK
+Wire Wire Line
+	6400 7700 5500 7700
+Wire Wire Line
+	5500 7700 5500 6400
 Wire Bus Line
 	10750 2150 10750 2350
@@
 	2750 1100 2750 1500
 Wire Bus Line
-	4700 6700 5400 6700
+	3900 6700 4600 6700
 Wire Bus Line
 	2650 1600 2650 2300
 Wire Bus Line
-	3100 6700 4600 6700
+	2300 6700 3800 6700
+Text GLabel 5900 1100 1    50   Input ~ 0
+6502_RDY_IN
 $EndSCHEMATC

Commit message: Added latch feature for EXRAM
Parts:
- J5: footprint Connector_PinHeader_2.54mm:PinHeader_2x12_P2.54mm_Vertical -> Connector_PinHeader_2.54mm:PinHeader_2x13_P2.54mm_Vertical; symbol Connector_Generic:Conn_02x12_Odd_Even -> Connector_Generic:Conn_02x13_Odd_Even
- R2: footprint Resistor_THT:R_Axial_DIN0207_L6.3mm_D2.5mm_P10.16mm_Horizontal -> Resistor_SMD:R_1206_3216Metric_Pad1.42x1.75mm_HandSolder
Connections:
- net 6502_RDY: now also J2.28 (Pin_28); no longer J2.26 (Pin_26)
- net DBG_WAIT: now also J2.27 (Pin_27); no longer J2.25 (Pin_25)
- net EXRAM: now also J5.26 (Pin_26)
- net IN12: now also J2.35 (Pin_35); no longer J2.33 (Pin_33)
- net IO13: now also J2.34 (Pin_34); no longer J2.32 (Pin_32)
- net IO14: now also J2.33 (Pin_33); no longer J2.31 (Pin_31)
- net IO15: now also J2.32 (Pin_32); no longer J2.30 (Pin_30)
- net IO16: now also J2.31 (Pin_31); no longer J2.29 (Pin_29)
- net IOCS: now also J2.23 (Pin_23); no longer J2.21 (Pin_21)
- net RDY_M1F: now also J2.24 (Pin_24); no longer J2.22 (Pin_22)
- net RDY_M2F: now also J2.25 (Pin_25); no longer J2.23 (Pin_23)
- net WS_DISABLE: now also J2.26 (Pin_26); no longer J2.24 (Pin_24)
- net ~PLD_RD: now also J2.29 (Pin_29); no longer J2.27 (Pin_27)
- net ~PLD_WR: now also J2.30 (Pin_30); no longer J2.28 (Pin_28)
- net LATCH_CP: now reaches J2.36 (Pin_36)
- new net LATCH_Q7: J5.25 (Pin_25)
- new net ~UART: J2.21 (Pin_21)
- new net ~VIA1: J2.22 (Pin_22)
Changed lines of the file:
@@
 Wire Wire Line
 	5600 7550 5600 6400
-Text GLabel 4350 5000 3    50   Input ~ 0
+Text GLabel 4650 5000 3    50   Input ~ 0
 RDY_M1F
-Text GLabel 4450 5000 3    50   Input ~ 0
+Text GLabel 4750 5000 3    50   Input ~ 0
 RDY_M2F
-Text GLabel 4550 5000 3    50   Input ~ 0
+Text GLabel 4850 5000 3    50   Input ~ 0
 WS_DISABLE
-Text GLabel 4650 5000 3    50   Input ~ 0
+Text GLabel 4950 5000 3    50   Input ~ 0
 DBG_WAIT
-Text GLabel 4750 5000 3    50   Output ~ 0
+Text GLabel 5050 5000 3    50   Output ~ 0
 6502_RDY
 Wire Wire Line
@@
 F 0 "R2" H 9920 1046 50  0000 L CNN
 F 1 "470" H 9920 955 50  0000 L CNN
-F 2 "Resistor_THT:R_Axial_DIN0207_L6.3mm_D2.5mm_P10.16mm_Horizontal" V 9780 1000 50  0001 C CNN
+F 2 "Resistor_SMD:R_1206_3216Metric_Pad1.42x1.75mm_HandSolder" V 9780 1000 50  0001 C CNN
 F 3 "~" H 9850 1000 50  0001 C CNN
 	1    9850 1000
@@
 	6650 900  6650 1100
 $Comp
-L Connector_Generic:Conn_02x12_Odd_Even J5
+L Connector_Generic:Conn_02x13_Odd_Even J5
 U 1 1 606B3BDC
-P 8650 1850
-F 0 "J5" H 8700 2567 50  0000 C CNN
-F 1 "JPR" H 8700 2476 50  0000 C CNN
-F 2 "Connector_PinHeader_2.54mm:PinHeader_2x12_P2.54mm_Vertical" H 8650 1850 50  0001 C CNN
-F 3 "~" H 8650 1850 50  0001 C CNN
-	1    8650 1850
+P 8650 1950
+F 0 "J5" H 8700 2750 50  0000 C CNN
+F 1 "JPR" H 8700 2650 50  0000 C CNN
+F 2 "Connector_PinHeader_2.54mm:PinHeader_2x13_P2.54mm_Vertical" H 8650 1950 50  0001 C CNN
+F 3 "~" H 8650 1950 50  0001 C CNN
+	1    8650 1950
 	1    0    0    -1
 $EndComp
@@
 	-1   0    0    1
 $EndComp
-Text GLabel 5050 5000 3    50   Input ~ 0
+Text GLabel 5350 5000 3    50   Input ~ 0
 ~PLD_WR
-Text GLabel 4900 5000 3    50   Input ~ 0
+Text GLabel 5200 5000 3    50   Input ~ 0
 ~PLD_RD
 Text GLabel 4100 5000 3    50   Input ~ 0
@@
 Text GLabel 4250 1100 1    50   Input ~ 0
 ROM_~CS
-Text GLabel 4250 5000 3    50   Input ~ 0
+Text GLabel 4550 5000 3    50   Input ~ 0
 IOCS
 Wire Wire Line
@@
 Wire Wire Line
 	4100 2800 6850 2800
-Text GLabel 5200 5000 3    50   Input ~ 0
+Text GLabel 5500 5000 3    50   Input ~ 0
 IO16
-Text GLabel 5300 5000 3    50   Input ~ 0
+Text GLabel 5600 5000 3    50   Input ~ 0
 IO15
-Text GLabel 5400 5000 3    50   Input ~ 0
+Text GLabel 5700 5000 3    50   Input ~ 0
 IO14
-Text GLabel 5500 5000 3    50   Input ~ 0
+Text GLabel 5800 5000 3    50   Input ~ 0
 IO13
-Text GLabel 5600 5000 3    50   Output ~ 0
+Text GLabel 5900 5000 3    50   Output ~ 0
 IN12
 Wire Wire Line
@@
 	4250 3000 6850 3000
 Wire Wire Line
-	4350 5000 4350 3100
-Wire Wire Line
-	4350 3100 6850 3100
-Wire Wire Line
-	4450 5000 4450 3200
-Wire Wire Line
-	4450 3200 6850 3200
-Wire Wire Line
-	4550 5000 4550 3300
-Wire Wire Line
-	4550 3300 6850 3300
-Wire Wire Line
-	4650 5000 4650 3400
-Wire Wire Line
-	4650 3400 6850 3400
-Wire Wire Line
-	4750 5000 4750 3500
-Wire Wire Line
-	4750 3500 6850 3500
-Wire Wire Line
-	4900 5000 4900 3600
-Wire Wire Line
-	4900 3600 6850 3600
+	4400 5000 4400 3100
+Wire Wire Line
+	4400 3100 6850 3100
+Wire Wire Line
+	4550 5000 4550 3200
+Wire Wire Line
+	4550 3200 6850 3200
+Wire Wire Line
+	4650 5000 4650 3300
+Wire Wire Line
+	4650 3300 6850 3300
+Wire Wire Line
+	4750 5000 4750 3400
+Wire Wire Line
+	4750 3400 6850 3400
+Wire Wire Line
+	4850 5000 4850 3500
+Wire Wire Line
+	4850 3500 6850 3500
+Wire Wire Line
+	4950 5000 4950 3600
+Wire Wire Line
+	4950 3600 6850 3600
 Wire Wire Line
 	5050 5000 5050 3700
@@
 	5200 3800 6850 3800
 Wire Wire Line
-	5300 5000 5300 3900
-Wire Wire Line
-	5300 3900 6850 3900
-Wire Wire Line
-	5400 5000 5400 4000
-Wire Wire Line
-	5400 4000 6850 4000
-Wire Wire Line
-	5500 5000 5500 4100
-Wire Wire Line
-	5500 4100 6850 4100
-Wire Wire Line
-	5600 5000 5600 4200
-Wire Wire Line
-	5600 4200 6850 4200
+	5350 5000 5350 3900
+Wire Wire Line
+	5350 3900 6850 3900
+Wire Wire Line
+	5500 5000 5500 4000
+Wire Wire Line
+	5500 4000 6850 4000
+Wire Wire Line
+	5600 5000 5600 4100
+Wire Wire Line
+	5600 4100 6850 4100
+Wire Wire Line
+	5700 5000 5700 4200
+Wire Wire Line
+	5700 4200 6850 4200
 Text GLabel 1650 4600 3    50   Output ~ 0
 ~NMI
@@
 Wire Wire Line
 	5500 7700 5500 6400
+Text GLabel 5900 1100 1    50   Input ~ 0
+6502_RDY_IN
+Text GLabel 4250 5000 3    50   Input ~ 0
+~UART
+Text GLabel 4400 5000 3    50   Input ~ 0
+~VIA1
+Wire Wire Line
+	5800 5000 5800 4300
+Wire Wire Line
+	5800 4300 6850 4300
+Wire Wire Line
+	5900 5000 5900 4400
+Wire Wire Line
+	5900 4400 6850 4400
+Text GLabel 6000 5000 3    50   Input ~ 0
+LATCH_CP
+Wire Wire Line
+	6000 5000 6000 4500
+Wire Wire Line
+	6000 4500 6850 4500
+Text GLabel 8250 2550 0    50   Input ~ 0
+LATCH_Q7
+Wire Wire Line
+	8250 2550 8450 2550
+Text GLabel 9150 2550 2    50   Output ~ 0
+EXRAM
+Wire Wire Line
+	8950 2550 9150 2550
 Wire Bus Line
 	10750 2150 10750 2350
@@
 Wire Bus Line
 	2300 6700 3800 6700
-Text GLabel 5900 1100 1    50   Input ~ 0
-6502_RDY_IN
 $EndSCHEMATC

Commit message: PCB Initial draft (no errors in DRC)
Parts:
- R10, R6, R7, R8, R9: footprint Resistor_THT:R_Axial_DIN0207_L6.3mm_D2.5mm_P10.16mm_Horizontal -> Resistor_SMD:R_1206_3216Metric_Pad1.42x1.75mm_HandSolder
Connections:
- net ~LATCH is gone; now on net ~VIA2: J9.17 (Pin_17)
- net 6502_CLK: now also J9.25 (Pin_25); no longer J9.26 (Pin_26)
- net LATCH_Q7: now also J9.40 (Pin_40)
- net R~W: now also J9.24 (Pin_24); no longer J9.25 (Pin_25)
- net ~6502_CLK: now also J9.26 (Pin_26); no longer J9.27 (Pin_27)
- net ~6502_RES: now also J9.27 (Pin_27); no longer J9.28 (Pin_28)
- net ~EXT_IRQ: now also J9.29 (Pin_29); no longer J9.30 (Pin_30)
- net ~IOCS0: now also J9.18 (Pin_18); no longer J9.19 (Pin_19)
- net ~IOCS1: now also J9.19 (Pin_19); no longer J9.20 (Pin_20)
- net ~IOCS2: now also J9.20 (Pin_20); no longer J9.21 (Pin_21)
- net ~IOCS3: now also J9.21 (Pin_21); no longer J9.22 (Pin_22)
- net ~NMI: now also J9.30 (Pin_30); no longer J9.31 (Pin_31)
- net ~RD: now also J9.22 (Pin_22); no longer J9.23 (Pin_23)
- net ~VIA2: no longer J9.18 (Pin_18)
- net ~VIA2_IRQ: now also J9.28 (Pin_28); no longer J9.29 (Pin_29)
- net ~WR: now also J9.23 (Pin_23); no longer J9.24 (Pin_24)
- net LATCH_Q0: now reaches J9.33 (Pin_33)
- net LATCH_Q1: now reaches J9.34 (Pin_34)
- net LATCH_Q2: now reaches J9.35 (Pin_35)
- net LATCH_Q3: now reaches J9.36 (Pin_36)
- net LATCH_Q4: now reaches J9.37 (Pin_37)
- net LATCH_Q5: now reaches J9.38 (Pin_38)
- net LATCH_Q6: now reaches J9.39 (Pin_39)
Changed lines of the file:
@@
 	2750 1500 2850 1600
 Text GLabel 2400 2400 1    50   Input ~ 0
-~LATCH
+~VIA2
 Text GLabel 2250 2400 1    50   Input ~ 0
-~VIA2
+~IOCS0
 Text GLabel 2100 2400 1    50   Input ~ 0
-~IOCS0
+~IOCS1
 Text GLabel 1950 2400 1    50   Input ~ 0
-~IOCS1
+~IOCS2
 Text GLabel 1800 2400 1    50   Input ~ 0
-~IOCS2
+~IOCS3
+Wire Wire Line
+	2400 2400 2400 2600
+Wire Wire Line
+	2400 2600 3050 2600
+Wire Wire Line
+	2250 2400 2250 2700
+Wire Wire Line
+	2250 2700 3050 2700
+Wire Wire Line
+	2100 2400 2100 2800
+Wire Wire Line
+	2100 2800 3050 2800
+Wire Wire Line
+	1950 2400 1950 2900
+Wire Wire Line
+	1950 2900 3050 2900
+Wire Wire Line
+	1800 2400 1800 3000
+Wire Wire Line
+	1800 3000 3050 3000
+Wire Wire Line
+	1650 2400 1650 3100
+Wire Wire Line
+	1650 3100 3050 3100
+Wire Wire Line
+	1500 2400 1500 3200
+Wire Wire Line
+	1500 3200 3050 3200
+Wire Wire Line
+	1350 2400 1350 3300
+Wire Wire Line
+	1350 3300 3050 3300
+Wire Wire Line
+	2550 2400 2550 2500
+Wire Wire Line
+	2550 2500 3050 2500
 Text GLabel 1650 2400 1    50   Input ~ 0
-~IOCS3
-Wire Wire Line
-	2400 2400 2400 2600
-Wire Wire Line
-	2400 2600 3050 2600
-Wire Wire Line
-	2250 2400 2250 2700
-Wire Wire Line
-	2250 2700 3050 2700
-Wire Wire Line
-	2100 2400 2100 2800
-Wire Wire Line
-	2100 2800 3050 2800
-Wire Wire Line
-	1950 2400 1950 2900
-Wire Wire Line
-	1950 2900 3050 2900
-Wire Wire Line
-	1800 2400 1800 3000
-Wire Wire Line
-	1800 3000 3050 3000
-Wire Wire Line
-	1650 2400 1650 3100
-Wire Wire Line
-	1650 3100 3050 3100
-Wire Wire Line
-	1500 2400 1500 3200
-Wire Wire Line
-	1500 3200 3050 3200
-Wire Wire Line
-	1350 2400 1350 3300
-Wire Wire Line
-	1350 3300 3050 3300
-Wire Wire Line
-	2550 2400 2550 2500
-Wire Wire Line
-	2550 2500 3050 2500
+~RD
 Text GLabel 1500 2400 1    50   Input ~ 0
-~RD
-Text GLabel 1350 2400 1    50   Input ~ 0
 ~WR
 Wire Wire Line
@@
 Wire Wire Line
 	5700 7400 5700 6400
-Text GLabel 1050 2400 1    50   Input ~ 0
+Text GLabel 1200 2400 1    50   Input ~ 0
 6502_CLK
 Wire Wire Line
@@
 Wire Wire Line
 	1350 3800 3050 3800
-Text GLabel 1200 2400 1    50   Input ~ 0
+Text GLabel 1350 2400 1    50   Input ~ 0
 R~W
 Wire Wire Line
@@
 Wire Wire Line
 	1200 3700 3050 3700
-Text GLabel 1200 4600 3    50   Input ~ 0
+Text GLabel 1050 4600 3    50   Input ~ 0
 ~6502_RES
 Wire Wire Line
@@
 F 0 "R10" V 10100 3850 50  0000 C CNN
 F 1 "27" V 10000 3850 50  0000 C CNN
-F 2 "Resistor_THT:R_Axial_DIN0207_L6.3mm_D2.5mm_P10.16mm_Horizontal" V 9930 3850 50  0001 C CNN
+F 2 "Resistor_SMD:R_1206_3216Metric_Pad1.42x1.75mm_HandSolder" V 9930 3850 50  0001 C CNN
 F 3 "~" H 10000 3850 50  0001 C CNN
 	1    10000 3850
@@
 F 0 "R9" V 10100 3600 50  0000 C CNN
 F 1 "27" V 10000 3600 50  0000 C CNN
-F 2 "Resistor_THT:R_Axial_DIN0207_L6.3mm_D2.5mm_P10.16mm_Horizontal" V 9930 3600 50  0001 C CNN
+F 2 "Resistor_SMD:R_1206_3216Metric_Pad1.42x1.75mm_HandSolder" V 9930 3600 50  0001 C CNN
 F 3 "~" H 10000 3600 50  0001 C CNN
 	1    10000 3600
@@
 F 0 "R7" V 8900 3400 50  0000 C CNN
 F 1 "4K7" V 9000 3400 50  0000 C CNN
-F 2 "Resistor_THT:R_Axial_DIN0207_L6.3mm_D2.5mm_P10.16mm_Horizontal" V 8930 3400 50  0001 C CNN
+F 2 "Resistor_SMD:R_1206_3216Metric_Pad1.42x1.75mm_HandSolder" V 8930 3400 50  0001 C CNN
 F 3 "~" H 9000 3400 50  0001 C CNN
 	1    9000 3400
@@
 F 0 "R8" V 9400 3400 50  0000 C CNN
 F 1 "10K" V 9500 3400 50  0000 C CNN
-F 2 "Resistor_THT:R_Axial_DIN0207_L6.3mm_D2.5mm_P10.16mm_Horizontal" V 9430 3400 50  0001 C CNN
+F 2 "Resistor_SMD:R_1206_3216Metric_Pad1.42x1.75mm_HandSolder" V 9430 3400 50  0001 C CNN
 F 3 "~" H 9500 3400 50  0001 C CNN
 	1    9500 3400
@@
 Wire Wire Line
 	2950 1000 3050 1000
+Text GLabel 1200 4600 3    50   Output ~ 0
+~VIA2_IRQ
 Text GLabel 1350 4600 3    50   Output ~ 0
-~VIA2_IRQ
-Text GLabel 1500 4600 3    50   Output ~ 0
 ~EXT_IRQ
 Wire Wire Line
-	1950 4600 1950 4200
-Wire Wire Line
-	1950 4200 3050 4200
-Wire Wire Line
-	2100 4600 2100 4300
-Wire Wire Line
-	2100 4300 3050 4300
+	2250 5000 2250 4200
+Wire Wire Line
+	2250 4200 3050 4200
+Wire Wire Line
+	2350 5000 2350 4300
+Wire Wire Line
+	2350 4300 3050 4300
 Text GLabel 6650 900  1    50   Input ~ 0
 GND
@@
 F 0 "R6" H 7680 4654 50  0000 R CNN
 F 1 "4K7" H 7680 4745 50  0000 R CNN
-F 2 "Resistor_THT:R_Axial_DIN0207_L6.3mm_D2.5mm_P10.16mm_Horizontal" V 7680 4700 50  0001 C CNN
+F 2 "Resistor_SMD:R_1206_3216Metric_Pad1.42x1.75mm_HandSolder" V 7680 4700 50  0001 C CNN
 F 3 "~" H 7750 4700 50  0001 C CNN
 	1    7750 4700
@@
 Wire Wire Line
 	5700 4200 6850 4200
-Text GLabel 1650 4600 3    50   Output ~ 0
+Text GLabel 1500 4600 3    50   Output ~ 0
 ~NMI
 Text GLabel 6500 1100 1    50   Input ~ 0
@@
 Text GLabel 6350 1100 1    50   Input ~ 0
 SYNC
-Text GLabel 1050 4600 3    50   Input ~ 0
+Text GLabel 1050 2400 1    50   Input ~ 0
 ~6502_CLK
 Text GLabel 6400 7700 2    50   Input ~ 0
@@
 Wire Wire Line
 	8950 2550 9150 2550
+Text GLabel 2950 5000 3    50   Input ~ 0
+LATCH_Q7
+Text GLabel 2850 5000 3    50   Input ~ 0
+LATCH_Q6
+Text GLabel 2750 5000 3    50   Input ~ 0
+LATCH_Q5
+Text GLabel 2650 5000 3    50   Input ~ 0
+LATCH_Q4
+Text GLabel 2550 5000 3    50   Input ~ 0
+LATCH_Q3
+Text GLabel 2450 5000 3    50   Input ~ 0
+LATCH_Q2
+Text GLabel 2350 5000 3    50   Input ~ 0
+LATCH_Q1
+Text GLabel 2250 5000 3    50   Input ~ 0
+LATCH_Q0
+Wire Wire Line
+	2950 5000 2950 4900
+Wire Wire Line
+	2950 4900 3050 4900
+Wire Wire Line
+	2850 5000 2850 4800
+Wire Wire Line
+	2850 4800 3050 4800
+Wire Wire Line
+	2750 5000 2750 4700
+Wire Wire Line
+	2750 4700 3050 4700
+Wire Wire Line
+	2650 5000 2650 4600
+Wire Wire Line
+	2650 4600 3050 4600
+Wire Wire Line
+	2550 5000 2550 4500
+Wire Wire Line
+	2550 4500 3050 4500
+Wire Wire Line
+	2450 5000 2450 4400
+Wire Wire Line
+	2450 4400 3050 4400
 Wire Bus Line
 	10750 2150 10750 2350
