File: Schematics/DB6502_proto/DB6502_proto.sch (KiCad schematic (older format))
At the start: 32 parts, among them U1 71256, U2 71256, U3 28C256, U4 65C02S, U5 74AC74, U6 74AC138, U7 22V10C, U8 74AC04, U9 74HC21

Commit message: Increased capacitor footprints to 1206
Parts:
- C1, C2, C3, C4, C5, C6, C8, C9: footprint Capacitor_SMD:C_0805_2012Metric_Pad1.15x1.40mm_HandSolder -> Capacitor_SMD:C_1206_3216Metric_Pad1.42x1.75mm_HandSolder
Changed lines of the file:
@@
 F 0 "C4" H 992 2196 50  0000 L CNN
 F 1 "0,1uF" H 992 2105 50  0000 L CNN
-F 2 "Capacitor_SMD:C_0805_2012Metric_Pad1.15x1.40mm_HandSolder" H 900 2150 50  0001 C CNN
+F 2 "Capacitor_SMD:C_1206_3216Metric_Pad1.42x1.75mm_HandSolder" H 900 2150 50  0001 C CNN
 F 3 "~" H 900 2150 50  0001 C CNN
 	1    900  2150
@@
 F 0 "C6" V 7121 3750 50  0000 C CNN
 F 1 "0,1uF" V 7212 3750 50  0000 C CNN
-F 2 "Capacitor_SMD:C_0805_2012Metric_Pad1.15x1.40mm_HandSolder" H 7350 3750 50  0001 C CNN
+F 2 "Capacitor_SMD:C_1206_3216Metric_Pad1.42x1.75mm_HandSolder" H 7350 3750 50  0001 C CNN
 F 3 "~" H 7350 3750 50  0001 C CNN
 	1    7350 3750
@@
 F 0 "C5" V 8821 3700 50  0000 C CNN
 F 1 "0,1uF" V 8912 3700 50  0000 C CNN
-F 2 "Capacitor_SMD:C_0805_2012Metric_Pad1.15x1.40mm_HandSolder" H 9050 3700 50  0001 C CNN
+F 2 "Capacitor_SMD:C_1206_3216Metric_Pad1.42x1.75mm_HandSolder" H 9050 3700 50  0001 C CNN
 F 3 "~" H 9050 3700 50  0001 C CNN
 	1    9050 3700
@@
 F 0 "C8" H 1392 7046 50  0000 L CNN
 F 1 "0,1uF" H 1392 6955 50  0000 L CNN
-F 2 "Capacitor_SMD:C_0805_2012Metric_Pad1.15x1.40mm_HandSolder" H 1300 7000 50  0001 C CNN
+F 2 "Capacitor_SMD:C_1206_3216Metric_Pad1.42x1.75mm_HandSolder" H 1300 7000 50  0001 C CNN
 F 3 "~" H 1300 7000 50  0001 C CNN
 	1    1300 7000
@@
 F 0 "C9" H 2292 7046 50  0000 L CNN
 F 1 "0,1uF" H 2292 6955 50  0000 L CNN
-F 2 "Capacitor_SMD:C_0805_2012Metric_Pad1.15x1.40mm_HandSolder" H 2200 7000 50  0001 C CNN
+F 2 "Capacitor_SMD:C_1206_3216Metric_Pad1.42x1.75mm_HandSolder" H 2200 7000 50  0001 C CNN
 F 3 "~" H 2200 7000 50  0001 C CNN
 	1    2200 7000
@@
 F 0 "C1" V 5021 1000 50  0000 C CNN
 F 1 "0,1uF" V 5112 1000 50  0000 C CNN
-F 2 "Capacitor_SMD:C_0805_2012Metric_Pad1.15x1.40mm_HandSolder" H 5250 1000 50  0001 C CNN
+F 2 "Capacitor_SMD:C_1206_3216Metric_Pad1.42x1.75mm_HandSolder" H 5250 1000 50  0001 C CNN
 F 3 "~" H 5250 1000 50  0001 C CNN
 	1    5250 1000
@@
 F 0 "C2" V 7371 1000 50  0000 C CNN
 F 1 "0,1uF" V 7462 1000 50  0000 C CNN
-F 2 "Capacitor_SMD:C_0805_2012Metric_Pad1.15x1.40mm_HandSolder" H 7600 1000 50  0001 C CNN
+F 2 "Capacitor_SMD:C_1206_3216Metric_Pad1.42x1.75mm_HandSolder" H 7600 1000 50  0001 C CNN
 F 3 "~" H 7600 1000 50  0001 C CNN
 	1    7600 1000
@@
 F 0 "C3" V 9771 1000 50  0000 C CNN
 F 1 "0,1uF" V 9862 1000 50  0000 C CNN
-F 2 "Capacitor_SMD:C_0805_2012Metric_Pad1.15x1.40mm_HandSolder" H 10000 1000 50  0001 C CNN
+F 2 "Capacitor_SMD:C_1206_3216Metric_Pad1.42x1.75mm_HandSolder" H 10000 1000 50  0001 C CNN
 F 3 "~" H 10000 1000 50  0001 C CNN
 	1    10000 1000

Commit message: Updates and fixes
Parts:
- JP1: footprint Connector_PinSocket_2.54mm:PinSocket_1x03_P2.54mm_Vertical -> Connector_PinHeader_2.54mm:PinHeader_1x03_P2.54mm_Vertical
Changed lines of the file:
@@
 F 0 "JP1" H 4750 3574 50  0000 C CNN
 F 1 "PLD CLK Selector" H 4750 3483 50  0000 C CNN
-F 2 "Connector_PinSocket_2.54mm:PinSocket_1x03_P2.54mm_Vertical" H 4750 3350 50  0001 C CNN
+F 2 "Connector_PinHeader_2.54mm:PinHeader_1x03_P2.54mm_Vertical" H 4750 3350 50  0001 C CNN
 F 3 "~" H 4750 3350 50  0001 C CNN
 	1    4750 3350

Commit message: Redesigned jumpers, introduced resistor network
Parts:
- removed JP2: PLD ~WR, Connector_PinHeader_2.54mm:PinHeader_1x02_P2.54mm_Vertical, symbol Jumper:Jumper_2_Open
- removed JP3: PLD ~RD, Connector_PinHeader_2.54mm:PinHeader_1x02_P2.54mm_Vertical, symbol Jumper:Jumper_2_Open
- removed JP4: PLD RDY, Connector_PinHeader_2.54mm:PinHeader_1x02_P2.54mm_Vertical, symbol Jumper:Jumper_2_Open
- removed JP5: PLD DBG_WAIT, Connector_PinHeader_2.54mm:PinHeader_1x02_P2.54mm_Vertical, symbol Jumper:Jumper_2_Open
- removed JP6: PLD WS_DISABLE, Connector_PinHeader_2.54mm:PinHeader_1x02_P2.54mm_Vertical, symbol Jumper:Jumper_2_Open
- removed JP7: PLD RDY_M1F, Connector_PinHeader_2.54mm:PinHeader_1x02_P2.54mm_Vertical, symbol Jumper:Jumper_2_Open
- removed JP8: PLD RDY_M2F, Connector_PinHeader_2.54mm:PinHeader_1x02_P2.54mm_Vertical, symbol Jumper:Jumper_2_Open
- removed R2, R3, R4: 4K7, Resistor_THT:R_Axial_DIN0207_L6.3mm_D2.5mm_P10.16mm_Horizontal, symbol Device:R
- added RN1: 4K7, Resistor_THT:R_Array_SIP5, symbol Device:R_Network04
Connections:
- net labels removed: DBG_WAIT, WS_DISABLE
- wire segments 323 -> 309
Changed lines of the file:
@@
 Text GLabel 7550 4950 2    50   Input ~ 0
 IO13
-Text GLabel 5050 5550 2    50   Input ~ 0
-WS_DISABLE
 Text GLabel 7550 4750 2    50   Input ~ 0
 IO15
@@
 Wire Wire Line
 	5100 7450 5650 7450
-$Comp
-L Device:R R2
-U 1 1 5FC6DB04
-P 4550 7000
-F 0 "R2" V 4450 7000 50  0000 C CNN
-F 1 "4K7" V 4550 7000 50  0000 C CNN
-F 2 "Resistor_THT:R_Axial_DIN0207_L6.3mm_D2.5mm_P10.16mm_Horizontal" V 4480 7000 50  0001 C CNN
-F 3 "~" H 4550 7000 50  0001 C CNN
-	1    4550 7000
-	1    0    0    -1
-$EndComp
-Text GLabel 4550 6800 1    50   Input ~ 0
+Text GLabel 4450 6550 1    50   Input ~ 0
 +5V
-Wire Wire Line
-	4550 6800 4550 6850
-Wire Wire Line
-	4550 7450 5100 7450
-Connection ~ 5100 7450
 Text GLabel 2850 7150 0    50   Input ~ 0
 GND
@@
 Wire Wire Line
 	1850 6550 1850 6600
-$Comp
-L Device:R R3
-U 1 1 6011A69F
-P 4750 7000
-F 0 "R3" V 4650 7000 50  0000 C CNN
-F 1 "4K7" V 4750 7000 50  0000 C CNN
-F 2 "Resistor_THT:R_Axial_DIN0207_L6.3mm_D2.5mm_P10.16mm_Horizontal" V 4680 7000 50  0001 C CNN
-F 3 "~" H 4750 7000 50  0001 C CNN
-	1    4750 7000
-	1    0    0    -1
-$EndComp
-Text GLabel 4750 6800 1    50   Input ~ 0
-+5V
-Wire Wire Line
-	4750 6800 4750 6850
-Wire Wire Line
-	4550 7150 4550 7450
-Wire Wire Line
-	4750 7150 4750 7350
-Wire Wire Line
-	4750 7350 5250 7350
-Connection ~ 5250 7350
 Wire Wire Line
 	7450 4550 8450 4550
@@
 Wire Wire Line
 	2150 5900 2250 5900
-$Comp
-L Jumper:Jumper_2_Open JP2
-U 1 1 604CBBF5
-P 4750 3950
-F 0 "JP2" H 4750 4185 50  0000 C CNN
-F 1 "PLD ~WR" H 4750 4094 50  0000 C CNN
-F 2 "Connector_PinHeader_2.54mm:PinHeader_1x02_P2.54mm_Vertical" H 4750 3950 50  0001 C CNN
-F 3 "~" H 4750 3950 50  0001 C CNN
-	1    4750 3950
-	1    0    0    -1
-$EndComp
-Text GLabel 4450 3950 0    50   Input ~ 0
-~PLD_WR
-Wire Wire Line
-	4450 3950 4550 3950
-Text GLabel 4450 4350 0    50   Input ~ 0
-~PLD_RD
-$Comp
-L Jumper:Jumper_2_Open JP3
-U 1 1 60561701
-P 4750 4350
-F 0 "JP3" H 4750 4597 50  0000 C CNN
-F 1 "PLD ~RD" H 4750 4499 50  0000 C CNN
-F 2 "Connector_PinHeader_2.54mm:PinHeader_1x02_P2.54mm_Vertical" H 4750 4350 50  0001 C CNN
-F 3 "~" H 4750 4350 50  0001 C CNN
-	1    4750 4350
-	1    0    0    -1
-$EndComp
-Wire Wire Line
-	4450 4350 4550 4350
-Text GLabel 5050 3950 2    50   Output ~ 0
-~WR
-Text GLabel 5050 4350 2    50   Output ~ 0
-~RD
-Wire Wire Line
-	4950 3950 5050 3950
-Wire Wire Line
-	4950 4350 5050 4350
-Text GLabel 4450 4750 0    50   Input ~ 0
-IO16
-$Comp
-L Jumper:Jumper_2_Open JP4
-U 1 1 605E4A7C
-P 4750 4750
-F 0 "JP4" H 4750 4985 50  0000 C CNN
-F 1 "PLD RDY" H 4750 4894 50  0000 C CNN
-F 2 "Connector_PinHeader_2.54mm:PinHeader_1x02_P2.54mm_Vertical" H 4750 4750 50  0001 C CNN
-F 3 "~" H 4750 4750 50  0001 C CNN
-	1    4750 4750
-	1    0    0    -1
-$EndComp
-Wire Wire Line
-	4450 4750 4550 4750
-Text GLabel 5050 4750 2    50   Output ~ 0
-6502_RDY
-Wire Wire Line
-	5050 4750 4950 4750
-$Comp
-L Device:R R4
-U 1 1 6068BEB8
-P 4950 7000
-F 0 "R4" V 4850 7000 50  0000 C CNN
-F 1 "4K7" V 4950 7000 50  0000 C CNN
-F 2 "Resistor_THT:R_Axial_DIN0207_L6.3mm_D2.5mm_P10.16mm_Horizontal" V 4880 7000 50  0001 C CNN
-F 3 "~" H 4950 7000 50  0001 C CNN
-	1    4950 7000
-	1    0    0    -1
-$EndComp
-Text GLabel 4950 6800 1    50   Input ~ 0
-+5V
-Wire Wire Line
-	4950 6800 4950 6850
-Wire Wire Line
-	4950 7150 4950 7250
-Wire Wire Line
-	4950 7250 5400 7250
-Connection ~ 5400 7250
-Text GLabel 5050 5150 2    50   Input ~ 0
-DBG_WAIT
-$Comp
-L Jumper:Jumper_2_Open JP5
-U 1 1 606CFBB5
-P 4750 5150
-F 0 "JP5" H 4750 5385 50  0000 C CNN
-F 1 "PLD DBG_WAIT" H 4750 5294 50  0000 C CNN
-F 2 "Connector_PinHeader_2.54mm:PinHeader_1x02_P2.54mm_Vertical" H 4750 5150 50  0001 C CNN
-F 3 "~" H 4750 5150 50  0001 C CNN
-	1    4750 5150
-	1    0    0    -1
-$EndComp
-Wire Wire Line
-	4450 5150 4550 5150
-Text GLabel 4450 5150 0    50   Output ~ 0
-IO15
-Wire Wire Line
-	4950 5150 5050 5150
-$Comp
-L Jumper:Jumper_2_Open JP6
-U 1 1 60715332
-P 4750 5550
-F 0 "JP6" H 4750 5785 50  0000 C CNN
-F 1 "PLD WS_DISABLE" H 4750 5694 50  0000 C CNN
-F 2 "Connector_PinHeader_2.54mm:PinHeader_1x02_P2.54mm_Vertical" H 4750 5550 50  0001 C CNN
-F 3 "~" H 4750 5550 50  0001 C CNN
-	1    4750 5550
-	1    0    0    -1
-$EndComp
-Wire Wire Line
-	4950 5550 5050 5550
 Text GLabel 7550 4850 2    50   Input ~ 0
 IO14
-Text GLabel 4450 5550 0    50   Output ~ 0
-IO14
-Wire Wire Line
-	4450 5550 4550 5550
-$Comp
-L Jumper:Jumper_2_Open JP7
-U 1 1 6077FFB1
-P 4750 5950
-F 0 "JP7" H 4750 6185 50  0000 C CNN
-F 1 "PLD RDY_M1F" H 4750 6094 50  0000 C CNN
-F 2 "Connector_PinHeader_2.54mm:PinHeader_1x02_P2.54mm_Vertical" H 4750 5950 50  0001 C CNN
-F 3 "~" H 4750 5950 50  0001 C CNN
-	1    4750 5950
-	1    0    0    -1
-$EndComp
-Wire Wire Line
-	4950 5950 5050 5950
-Text GLabel 4450 5950 0    50   Output ~ 0
-IO13
-Wire Wire Line
-	4450 5950 4550 5950
-$Comp
-L Jumper:Jumper_2_Open JP8
-U 1 1 607A3E01
-P 4750 6350
-F 0 "JP8" H 4750 6585 50  0000 C CNN
-F 1 "PLD RDY_M2F" H 4750 6494 50  0000 C CNN
-F 2 "Connector_PinHeader_2.54mm:PinHeader_1x02_P2.54mm_Vertical" H 4750 6350 50  0001 C CNN
-F 3 "~" H 4750 6350 50  0001 C CNN
-	1    4750 6350
-	1    0    0    -1
-$EndComp
-Wire Wire Line
-	4950 6350 5050 6350
-Text GLabel 4450 6350 0    50   Output ~ 0
-IN12
-Wire Wire Line
-	4450 6350 4550 6350
-Text GLabel 5050 5950 2    50   Input ~ 0
-RDY_M2F
-Text GLabel 5050 6350 2    50   Input ~ 0
-RDY_M1F
 Wire Wire Line
 	6350 3850 6350 3950
@@
 Text GLabel 6350 3850 1    50   Input ~ 0
 PLD_CLK
+$Comp
+L Device:R_Network04 RN1
+U 1 1 6054D542
+P 4650 6850
+F 0 "RN1" H 4838 6896 50  0000 L CNN
+F 1 "4K7" H 4838 6805 50  0000 L CNN
+F 2 "Resistor_THT:R_Array_SIP5" V 4925 6850 50  0001 C CNN
+F 3 "http://www.vishay.com/docs/31509/csc.pdf" H 4650 6850 50  0001 C CNN
+	1    4650 6850
+	1    0    0    -1
+$EndComp
+Wire Wire Line
+	4450 6550 4450 6650
+Wire Wire Line
+	4750 7050 4750 7150
+Wire Wire Line
+	4750 7150 5550 7150
+Connection ~ 5550 7150
+Wire Wire Line
+	4650 7050 4650 7250
+Wire Wire Line
+	4650 7250 5400 7250
+Connection ~ 5400 7250
+Wire Wire Line
+	4550 7050 4550 7350
+Wire Wire Line
+	4550 7350 5250 7350
+Connection ~ 5250 7350
+Wire Wire Line
+	4450 7050 4450 7450
+Wire Wire Line
+	4450 7450 5100 7450
+Connection ~ 5100 7450
 Wire Bus Line
 	8500 4150 8500 4350

Commit message: Working on a PCB
Parts:
- RN1: footprint Resistor_THT:R_Array_SIP5 -> Resistor_THT:R_Array_SIP9; symbol Device:R_Network04 -> Device:R_Network08
Connections:
- net BE: now also RN1.9 (R8)
- net ~NMI: now also RN1.8 (R7)
- net ~SO: now also RN1.7 (R6)
- new net SR_OUT: RN1.6 (R5)
Changed lines of the file:
@@
 Wire Wire Line
 	5100 7450 5650 7450
-Text GLabel 4450 6550 1    50   Input ~ 0
+Text GLabel 3800 5950 1    50   Input ~ 0
 +5V
 Text GLabel 2850 7150 0    50   Input ~ 0
@@
 PLD_CLK
 $Comp
-L Device:R_Network04 RN1
+L Device:R_Network08 RN1
 U 1 1 6054D542
-P 4650 6850
-F 0 "RN1" H 4838 6896 50  0000 L CNN
-F 1 "4K7" H 4838 6805 50  0000 L CNN
-F 2 "Resistor_THT:R_Array_SIP5" V 4925 6850 50  0001 C CNN
-F 3 "http://www.vishay.com/docs/31509/csc.pdf" H 4650 6850 50  0001 C CNN
-	1    4650 6850
-	1    0    0    -1
-$EndComp
-Wire Wire Line
-	4450 6550 4450 6650
-Wire Wire Line
-	4750 7050 4750 7150
-Wire Wire Line
-	4750 7150 5550 7150
+P 4200 6250
+F 0 "RN1" H 4600 6300 50  0000 L CNN
+F 1 "4K7" H 4600 6200 50  0000 L CNN
+F 2 "Resistor_THT:R_Array_SIP9" V 4475 6250 50  0001 C CNN
+F 3 "http://www.vishay.com/docs/31509/csc.pdf" H 4200 6250 50  0001 C CNN
+	1    4200 6250
+	1    0    0    -1
+$EndComp
+Wire Wire Line
+	3800 5950 3800 6050
+Wire Wire Line
+	4100 6450 4100 7150
+Wire Wire Line
+	4100 7150 5550 7150
 Connection ~ 5550 7150
 Wire Wire Line
-	4650 7050 4650 7250
-Wire Wire Line
-	4650 7250 5400 7250
+	4000 6450 4000 7250
+Wire Wire Line
+	4000 7250 5400 7250
 Connection ~ 5400 7250
 Wire Wire Line
-	4550 7050 4550 7350
-Wire Wire Line
-	4550 7350 5250 7350
+	3900 6450 3900 7350
+Wire Wire Line
+	3900 7350 5250 7350
 Connection ~ 5250 7350
 Wire Wire Line
-	4450 7050 4450 7450
-Wire Wire Line
-	4450 7450 5100 7450
+	3800 6450 3800 7450
+Wire Wire Line
+	3800 7450 5100 7450
 Connection ~ 5100 7450
+Text GLabel 4600 6550 2    50   Output ~ 0
+BE
+Wire Wire Line
+	4500 6550 4500 6450
+Text GLabel 4600 6700 2    50   Output ~ 0
+~NMI
+Wire Wire Line
+	4500 6550 4600 6550
+Wire Wire Line
+	4600 6700 4400 6700
+Wire Wire Line
+	4400 6700 4400 6450
+Text GLabel 4600 6850 2    50   Output ~ 0
+~SO
+Wire Wire Line
+	4300 6450 4300 6850
+Wire Wire Line
+	4300 6850 4600 6850
+Text GLabel 4600 7000 2    50   Output ~ 0
+SR_OUT
+Wire Wire Line
+	4600 7000 4200 7000
+Wire Wire Line
+	4200 7000 4200 6450
 Wire Bus Line
 	8500 4150 8500 4350

Commit message: Small fixes on PCB
Connections:
- net BE: no longer RN1.9 (R8)
Changed lines of the file:
@@
 	3800 7450 5100 7450
 Connection ~ 5100 7450
-Text GLabel 4600 6550 2    50   Output ~ 0
-BE
-Wire Wire Line
-	4500 6550 4500 6450
 Text GLabel 4600 6700 2    50   Output ~ 0
 ~NMI
 Wire Wire Line
-	4500 6550 4600 6550
-Wire Wire Line
 	4600 6700 4400 6700
